Commit message: Update README

File: scenario1/urdf/hand.urdf.xacro (robot description, xacro)
@@ -2,7 +2,7 @@
 <robot xmlns:xacro="http://www.ros.org/wiki/xacro" name="hand">
 	<xacro:include filename="$(find soft_hand_description)/model/soft_hand.urdf.xacro"/>
-		<link name="wrist"/>
-		<xacro:soft_hand parent="wrist" name="$(arg name)" withAdaptiveTransmission="true" useMimicTag="false" left="false">
-				<origin xyz="0.002 0.009 0.038" rpy="0 0 0"/>
+		<link name="hand"/>
+		<xacro:soft_hand parent="hand" name="$(arg name)" withAdaptiveTransmission="true" useMimicTag="false" left="false">
+				<origin xyz="0.0 0.0 0.0" rpy="0 0 0"/>
 		</xacro:soft_hand>
 </robot>
